Commit message: added support for gazebo and rviz simulation for 2wd and 4wd rovers

File: rr_openrover_description/urdf/2WD_rover.urdf.xacro (robot description, xacro)
@@ -2,21 +2,17 @@
 <robot name="2WD_rover" xmlns:xacro="http://ros.org/wiki/xacro">
   <xacro:include filename="$(find rr_openrover_description)/urdf/common_properties.xacro"/>
-  <xacro:include filename="$(find rr_openrover_description)/urdf/2WD_Rover.gazebo.xacro"/>
+  <xacro:include filename="$(find rr_openrover_description)/urdf/2WD_rover.gazebo.xacro"/>
   <link name="base_footprint"/>
+  <link name="base_link"/>
   <joint name="base_joint" type="fixed">
     <parent link="base_footprint"/>
     <child link="base_link"/>
-    <origin xyz="0 0 0.12" rpy="0 0 0"/>
+    <origin xyz="0 0 0" rpy="0 0 0"/>
   </joint>
-  <link name="base_link">
+  <link name="chassis_link">
     <visual>
-      <origin xyz="-0.142 0 0.055" rpy="0 0 1.57"/>
+      <origin xyz="0 0 0" rpy="${pi / 2} 0 ${pi / 2}"/>
       <geometry>
-        <mesh filename="package://rr_openrover_description/meshes/2WD_OpenRover.stl" scale="1 1 1"/>
-      <!--
-      <origin xyz="-0.142 0 0" rpy="0 0 0"/>
-      <geometry>
-        <box size="0.42 0.25 0.12"/>
-        -->
+        <mesh filename="package://rr_openrover_description/meshes/2WD_Rover/2WDCore.stl" scale="0.001 0.001 0.001"/>
       </geometry>
       <material name="dark"/>
@@ -31,258 +27,169 @@
       <origin xyz="-0.142 0 0" rpy="0 0 0" />
       <mass value="7.5" />
-      <inertia ixx="4.806e-2"
-               ixy="0.0" iyy="1.193e-1"
-               ixz="0.0" iyz="0.0" izz="1.493e-1" />
+      <inertia ixx="5.914e-2"
+               ixy="0.0" iyy="1.713e-1"
+               ixz="0.0" iyz="1.815e-3" izz="5.917e-2" />
     </inertial>
   </link>
-  <joint name="wheel_left_joint" type="continuous">
+  <joint name="chassis_joint" type="fixed">
     <parent link="base_link"/>
-    <child link="wheel_left_link"/>
-    <origin xyz="0 0.179 0" rpy="-1.57 0 0"/>
-    <axis xyz="0 0 1"/>
+    <child link="chassis_link"/>
+    <origin xyz="0 0 0.14" rpy="0 0 0"/>
   </joint>
-  <link name="wheel_left_link">
+  <link name="left_front_wheel_link">
     <visual>
-      <origin xyz="0 0 0" rpy="-1.57 0 0"/>
+      <origin xyz="0 -0.18 0" rpy="0 0 ${pi / 2}"/>
       <geometry>
-        <mesh filename="package://rr_openrover_description/meshes/left_wheel.stl" scale="1 1 1"/>
-      <!--
-      <origin xyz="0 0 0" rpy="0 0 3.14"/>
-      <geometry>
-        <cylinder length="0.07" radius="0.12"/>
-        -->
-      </geometry>
-      <material name="black"/>
-    </visual>
-    <collision>
-      <origin xyz="0 0 0" rpy="0 0 3.14"/>
-      <geometry>
-        <cylinder length="0.07" radius="0.12"/>
-      </geometry>
-    </collision>
-    <inertial>
-      <origin xyz="0 0 0" rpy="0 0 3.14" />
-      <mass value="1.525" />
-      <inertia ixx="6.723e-3"
-               ixy="0.0" iyy="6.723e-3"
-               ixz="0.0" iyz="0.0" izz="1.220e-2" />
-    </inertial>
-  </link>
-  <joint name="wheel_right_joint" type="continuous">
-    <parent link="base_link"/>
-    <child link="wheel_right_link"/>
-    <origin xyz="0 -0.179 0" rpy="-1.57 0 0"/>
-    <axis xyz="0 0 1"/>
-  </joint>
-  <link name="wheel_right_link">
-    <visual>
-      <origin xyz="0 0 0" rpy="1.57 0 0"/>
-      <geometry>
-        <mesh filename="package://rr_openrover_description/meshes/right_wheel.stl" scale="1 1 1"/>
-      <!--
-      <origin xyz="0 0 0" rpy="0 0 0"/>
-      <geometry>
-        <cylinder length="0.07" radius="0.12"/>
-        -->
-      </geometry>
-      <material name="black"/>
-    </visual>
-    <collision>
-      <origin xyz="0 0 0" rpy="0 0 0"/>
-      <geometry>
-        <cylinder length="0.07" radius="0.12"/>
-      </geometry>
-    </collision>
-    <inertial>
-      <origin xyz="0 0 0" rpy="0 0 0" />
-      <mass value="1.525" />
-      <inertia ixx="6.723e-3"
-               ixy="0.0" iyy="6.723e-3"
-               ixz="0.0" iyz="0.0" izz="1.220e-2" />
-    </inertial>
-  </link>
-  <joint name="sheetmetal_joint" type="fixed">
-    <parent link="base_link"/>
-    <child link="sheetmetal_link"/>
-    <origin xyz="-0.35 0 0" rpy="0 0 0"/>
-  </joint>
-  <link name="sheetmetal_link">
-    <visual>
-      <origin xyz="0 0 0" rpy="1.57 0 -1.57"/>
-      <geometry>
-        <mesh filename="package://rr_openrover_description/meshes/sheetmetal_part.stl" scale="1 1 1"/>
-      <!--
-      <origin xyz="0 0 0" rpy="0 0 0"/>
-      <geometry>
-        <box size="0.065 0.4 0.008"/>
-        -->
+        <mesh filename="package://rr_openrover_description/meshes/2WD_Rover/LeftFrontTire.stl" scale="0.001 0.001 0.001"/>
       </geometry>
       <material name="dark"/>
     </visual>
     <collision>
-      <origin xyz="-0.007 0 0" rpy="0 0 0"/>
+      <origin xyz="0 0 0" rpy="${pi / 2} 0 0"/>
       <geometry>
-        <box size="0.065 0.4 0.008"/>
+        <cylinder length="0.07" radius="0.127"/>
       </geometry>
     </collision>
     <inertial>
-      <origin xyz="0 0 0" />
-      <mass value="0.6" />
-      <inertia ixx="8.020e-3"
-               ixy="0.0" iyy="2.313e-4"
-               ixz="0.0" iyz="0.0" izz="8.211e-3" />
+      <origin xyz="0 0 0" rpy="0 0 0"/>
+      <mass value="0.25" />
+      <inertia ixx="7.75e-3"
+               ixy="0.0" iyy="1.713e-1"
+               ixz="0.0" iyz="1.815e-3" izz="5.917e-2" />
     </inertial>
   </link>
-  <joint name="plate_link_joint" type="fixed">
-    <parent link="base_link"/>
-    <child link="plate_link"/>
-    <origin xyz="-0.1365 0 0.127" rpy="0 0 0"/>
+  <joint name="left_front_wheel_joint" type="continuous">
+    <parent link="chassis_link"/>
+    <child link="left_front_wheel_link"/>
+    <origin xyz="0 0.18 0" rpy="0 0 0"/>
+    <axis xyz="0 1 0" rpy="0 0 0"/>
   </joint>
-  <link name="plate_link">
+  <link name="right_front_wheel_link">
     <visual>
-      <origin xyz="0 0 0" rpy="0 0 0"/>
+      <origin xyz="0 0.18 0" rpy="0 0 ${pi / 2}"/>
       <geometry>
-        <box size="0.381 0.254 0.005"/>
+        <mesh filename="package://rr_openrover_description/meshes/2WD_Rover/RightFrontTire.stl" scale="0.001 0.001 0.001"/>
       </geometry>
-      <material name="acrylic"/>
-    </visual>
-    <inertial>
-      <origin xyz="0 0 0" />
-      <mass value="0.65" />
-      <inertia ixx="3.496e-3"
-               ixy="0.0" iyy="7.864e-3"
-               ixz="0.0" iyz="0.0" izz="1.136e-2" />
-    </inertial>
-  </link>
-  <joint name="imu_link_joint" type="fixed">
-    <parent link="plate_link"/>
-    <child link="imu_link"/>
-    <origin xyz="0.1365 0 0.0026" rpy="0 0 0"/>
-  </joint>
-  <link name="imu_link">
-    <visual>
-      <origin xyz="0 0 0" rpy="0 0 0"/>
-      <geometry>
-        <box size="0.01 0.01 0.002"/>
-      </geometry>
-      <material name="blue"/>
-    </visual>
-    <inertial>
-      <origin xyz="0 0 0" />
-      <mass value="0.04" />
-      <inertia ixx="3.467e-7"
-               ixy="0.0" iyy="3.467e-7"
-               ixz="0.0" iyz="0.0" izz="6.667e-7" />
-    </inertial>
-  </link>
-  <joint name="cpu_link_joint" type="fixed">
-    <parent link="plate_link"/>
-    <child link="cpu_link"/>
-    <origin xyz="-0.0032 0 0.0275" rpy="0 0 0"/>
-  </joint>
-  <link name="cpu_link">
-    <visual>
-      <origin xyz="0 0 0" rpy="0 0 0"/>
-      <geometry>
-        <box size="0.111 0.117 0.05"/>
-      </geometry>
-      <material name="light_black"/>
-    </visual>
-    <inertial>
-      <origin xyz="0 0 0" />
-      <mass value="0.64" />
-      <inertia ixx="8.634e-4"
-               ixy="0.0" iyy="7.905e-4"
-               ixz="0.0" iyz="0.0" izz="1.387e-3" />
-    </inertial>
-  </link>
-  <joint name="lidar_link_joint" type="fixed">
-    <parent link="cpu_link"/>
-    <child link="lidar_link"/>
-    <origin xyz="0 0 0.0488" rpy="0 0 0"/>
-  </joint>
-  <link name="lidar_link">
-    <visual>
-      <origin xyz="0 0 0" rpy="0 0 0"/>
-      <geometry>
-        <cylinder length="0.0476" radius="0.0381"/>
-      </geometry>
-      <material name="light_black"/>
-    </visual>
-    <inertial>
-      <origin xyz="0 0 0" />
-      <mass value="0.220" />
-      <inertia ixx="1.214e-4"
-               ixy="0.0" iyy="1.214e-4"
-               ixz="0.0" iyz="0.0" izz="1.597e-4" />
-    </inertial>
-  </link>
-  <joint name="caster_back_left_joint" type="continuous">
-    <parent link="sheetmetal_link"/>
-    <child link="caster_back_left_link"/>
-    <origin xyz="-0.01 0.17 -0.01" rpy="0 0 0"/>
-    <axis xyz="0 0 1"/>
-    <dynamics damping="0.1" friction="0.01"/>
-  </joint>
-  <link name="caster_back_left_link">
-    <visual>
-      <origin xyz="0 0 0" rpy="1.57 0 3.14"/>
-      <geometry>
-        <mesh filename="package://rr_openrover_description/meshes/left_caster_wheel.stl" scale="1 1 1"/>
-      <!--
-      <origin xyz="-0.028 0 -0.065" rpy="1.57 0 3.14"/>
-      <geometry>
-        <cylinder length="0.035" radius="0.048"/>
-        -->
-      </geometry>
-      <material name="grey"/>
+      <material name="dark"/>
     </visual>
     <collision>
-      <origin xyz="-0.035 0 -0.065" rpy="1.57 0 3.14"/>
+      <origin xyz="0 0 0" rpy="${pi / 2} 0 0"/>
       <geometry>
-        <cylinder length="0.0035" radius="0.05"/>
+        <cylinder length="0.07" radius="0.127"/>
       </geometry>
     </collision>
     <inertial>
-      <origin xyz="-0.005 0 -0.03" />
-      <mass value="0.41" />
-      <inertia ixx="3.841e-4"
-               ixy="0.0" iyy="4.592e-4"
-               ixz="0.0" iyz="0.0" izz="2.135e-4" />
+      <origin xyz="0 0 0" rpy="0 0 0"/>
+      <mass value="0.25" />
+      <inertia ixx="7.750e-3"
+               ixy="0.0" iyy="4.546-3"
+               ixz="0.0" iyz="1.478e-8" izz="4.545-3" />
     </inertial>
   </link>
-  <joint name="caster_back_right_joint" type="continuous">
-    <parent link="sheetmetal_link"/>
-    <child link="caster_back_right_link"/>
-    <origin xyz="-0.01 -0.17 -0.01" rpy="0 0 0"/>
+  <joint name="right_front_wheel_joint" type="continuous">
+    <parent link="chassis_link"/>
+    <child link="right_front_wheel_link"/>
+    <origin xyz="0 -0.18 0" rpy="0 0 0"/>
+    <axis xyz="0 1 0"/>
+  </joint>
+  <link name="left_rear_castor_housing_link">
+    <visual>
+      <origin xyz="0.355 -0.171 0" rpy="${pi / 2} 0 ${pi / 2}"/>
+      <geometry>
+        <mesh filename="package://rr_openrover_description/meshes/2WD_Rover/LeftRearCastorHousing.stl" scale="0.001 0.001 0.001"/>
+      </geometry>ps -aux | grep gazebo | awk $2
+      <material name="dark"/>
+    </visual>
+    <inertial>
+      <origin xyz="0 0 0" rpy="0 0 0"/>
+      <mass value="0.25" />
+      <inertia ixx="4.81e-5"
+               ixy="0.0" iyy="2.939e-5"
+               ixz="0.0" iyz="1.478e-5" izz="4.914e-5" />
+    </inertial>
+  </link>
+  <joint name="left_rear_castor_housing_joint" type="continuous">
+    <parent link="chassis_link"/>
+    <child link="left_rear_castor_housing_link"/>
+    <origin xyz="-0.355 0.175 0.005" rpy="0 0 0"/>
     <axis xyz="0 0 1"/>
-    <dynamics damping="0.1" friction="0.01"/>
   </joint>
-  <link name="caster_back_right_link">
+  <link name="left_rear_castor_wheel_link">
     <visual>
-      <origin xyz="0 0 0" rpy="1.57 0 3.14"/>
+      <origin xyz="0.385 -0.170 0.083" rpy="${pi / 2} 0 ${pi / 2}"/>
       <geometry>
-        <mesh filename="package://rr_openrover_description/meshes/right_caster_wheel.stl" scale="1 1 1"/>
-      <!--
-      <origin xyz="-0.028 0 -0.065" rpy="1.57 0 3.14"/>
-      <geometry>
-        <cylinder length="0.035" radius="0.048"/>
-        -->
+        <mesh filename="package://rr_openrover_description/meshes/2WD_Rover/LeftRearCastorWheel.stl" scale="0.001 0.001 0.001"/>
       </geometry>
-      <material name="grey"/>
+      <material name="dark"/>
     </visual>
     <collision>
-      <origin xyz="-0.035 0 -0.065" rpy="1.57 0 3.14"/>
+      <origin xyz="0 0 0" rpy="${pi / 2} 0 0"/>
       <geometry>
-        <cylinder length="0.0035" radius="0.05"/>
+        <cylinder length="0.0254" radius="0.050"/>
       </geometry>
     </collision>
     <inertial>
-      <origin xyz="-0.005 0 -0.03" />
-      <mass value="0.41" />
-      <inertia ixx="3.841e-4"
-               ixy="0.0" iyy="4.592e-4"
-               ixz="0.0" iyz="0.0" izz="2.135e-4" />
+      <origin xyz="0 0 0" rpy="0 0 0"/>
+      <mass value="0.25" />
+      <inertia ixx="2.511e-4"
+               ixy="0.0" iyy="2.136-4"
+               ixz="0.0" iyz="1.478e-4" izz="1.363e-4" />
     </inertial>
   </link>
+  <joint name="left_rear_castor_wheel_joint" type="continuous">
+    <parent link="left_rear_castor_housing_link"/>
+    <child link="left_rear_castor_wheel_link"/>
+    <origin xyz="-0.028 0 -0.08" rpy="0 0 0"/>
+    <axis xyz="0 1 0"/>
+  </joint>
+  <link name="right_rear_castor_housing_link">
+    <visual>
+      <origin xyz="0.355 0.171 0" rpy="${pi / 2} 0 ${pi / 2}"/>
+      <geometry>
+        <mesh filename="package://rr_openrover_description/meshes/2WD_Rover/RightRearCastorHousing.stl" scale="0.001 0.001 0.001"/>
+      </geometry>
+      <material name="dark"/>
+    </visual>
+    <inertial>
+      <origin xyz="0 0 0" rpy="0 0 0"/>
+      <mass value="0.25" />
+      <inertia ixx="4.81e-5"
+               ixy="0.0" iyy="2.939e-5"
+               ixz="0.0" iyz="1.478e-5" izz="4.914e-5" />
+    </inertial>
+  </link>
+  <joint name="right_rear_castor_housing_joint" type="continuous">
+    <parent link="chassis_link"/>
+    <child link="right_rear_castor_housing_link"/>
+    <origin xyz="-0.355 -0.175 0.005" rpy="0 0 0"/>
+    <axis xyz="0 0 1"/>
+  </joint>
+  <link name="right_rear_castor_wheel_link">
+    <visual>
+      <origin xyz="0.385 0.171 0.083" rpy="${pi / 2} 0 ${pi / 2}"/>
+      <geometry>
+        <mesh filename="package://rr_openrover_description/meshes/2WD_Rover/RightRearCastorWheel.stl" scale="0.001 0.001 0.001"/>
+      </geometry>
+      <material name="dark"/>
+    </visual>
+    <collision>
+      <origin xyz="0 0 0" rpy="${pi / 2} 0 0"/>
+      <geometry>
+        <cylinder length="0.0254" radius="0.050"/>
+      </geometry>
+    </collision>
+    <inertial>
+      <origin xyz="0 0 0" rpy="0 0 0"/>
+      <mass value="0.25" />
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
File: rr_openrover_description/urdf/4WD_rover.urdf.xacro (robot description, xacro)
@@ -2,17 +2,19 @@
 <robot name="4WD_rover" xmlns:xacro="http://ros.org/wiki/xacro">
   <xacro:include filename="$(find rr_openrover_description)/urdf/common_properties.xacro"/>
+  <xacro:include filename="$(find rr_openrover_description)/urdf/4WD_rover.gazebo.xacro"/>
   <xacro:property name="PI" value="3.1415926535897931" />
   <xacro:property name="rover_4wd_ground_clearance" value="0.182" />
+  <link name="base_footprint"/>
   <link name="base_link"/>
-  <joint name="base_link_joint" type="fixed">
-    <parent link="base_link"/>
-    <child link="chassis_link"/>
+  <joint name="base_joint" type="fixed">
+    <parent link="base_footprint"/>
+    <child link="base_link"/>
     <origin xyz="0 0 0" rpy="0 0 0"/>
   </joint>
   <link name="chassis_link">
     <visual>
-      <origin xyz="0 0 ${rover_4wd_ground_clearance}" rpy="0 0 ${PI/2}"/>
+      <origin xyz="0 0 0" rpy="${pi / 2} 0 ${pi / 2}"/>
       <geometry>
-        <mesh filename="package://rr_openrover_description/meshes/4WD_OpenRover.stl" scale="1 1 1"/>
+        <mesh filename="package://rr_openrover_description/meshes/4WD_Rover/4WDCore.stl" scale="0.001 0.001 0.001"/>
       </geometry>
       <material name="dark"/>
@@ -27,9 +29,126 @@
       <origin xyz="-0.142 0 0" rpy="0 0 0" />
       <mass value="7.5" />
-      <inertia ixx="4.806e-2"
-               ixy="0.0" iyy="1.193e-1"
-               ixz="0.0" iyz="0.0" izz="1.493e-1" />
+      <inertia ixx="5.914e-5"
+               ixy="0.0" iyy="1.713e-4"
+               ixz="0.0" iyz="1.815e-6" izz="5.917e-5" />
     </inertial>
   </link>
-<xacro:include filename="$(find rr_openrover_description)/urdf/accessories.urdf.xacro" />
+  <joint name="chassis_joint" type="fixed">
+    <parent link="base_link"/>
+    <child link="chassis_link"/>
+    <origin xyz="0 0 0.127" rpy="0 0 0"/>
+  </joint>
+  <link name="left_front_wheel_link">
+    <visual>
+      <origin xyz="0 -0.18 0" rpy="0 0 ${pi / 2}"/>
+      <geometry>
+        <mesh filename="package://rr_openrover_description/meshes/4WD_Rover/LeftFrontWheel.stl" scale="0.001 0.001 0.001"/>
+      </geometry>
+      <material name="dark"/>
+    </visual>
+    <collision>
+      <origin xyz="0 0 0" rpy="${pi / 2} 0 0"/>
+      <geometry>
+        <cylinder length="0.07" radius="0.127"/>
+      </geometry>
+    </collision>
+    <inertial>
+      <origin xyz="0 0 0" rpy="0 0 0"/>
+      <mass value="0.25" />
+      <inertia ixx="7.750e-6"
+               ixy="0.0" iyy="4.546-6"
+               ixz="0.0" iyz="1.478e-8" izz="4.545-6" />
+    </inertial>
+  </link>
+  <joint name="left_front_wheel_joint" type="continuous">
+    <parent link="chassis_link"/>
+    <child link="left_front_wheel_link"/>
+    <origin xyz="0 0.18 0" rpy="0 0 0"/>
+    <axis xyz="0 1 0"/>
+  </joint>
+  <link name="right_front_wheel_link">
+    <visual>
+      <origin xyz="0 0.18 0" rpy="0 0 ${pi / 2}"/>
+      <geometry>
+        <mesh filename="package://rr_openrover_description/meshes/4WD_Rover/RightFrontWheel.stl" scale="0.001 0.001 0.001"/>
+      </geometry>
+      <material name="dark"/>
+    </visual>
+    <collision>
+      <origin xyz="0 0 0" rpy="${pi / 2} 0 0"/>
+      <geometry>
+        <cylinder length="0.07" radius="0.127"/>
+      </geometry>
+    </collision>
+    <inertial>
+      <origin xyz="0 0 0" rpy="0 0 0"/>
+      <mass value="0.25" />
+      <inertia ixx="7.750e-6"
+               ixy="0.0" iyy="4.546-6"
+               ixz="0.0" iyz="1.478e-8" izz="4.545-6" />
+    </inertial>
+  </link>
+  <joint name="right_front_wheel_joint" type="continuous">
+    <parent link="chassis_link"/>
+    <child link="right_front_wheel_link"/>
+    <origin xyz="0 -0.18 0" rpy="0 0 0"/>
+    <axis xyz="0 1 0"/>
+  </joint>
+  <link name="left_rear_wheel_link">
+    <visual>
+      <origin xyz="0.284 -0.18 0" rpy="${pi / 2} 0 ${pi / 2}"/>
+      <geometry>
+        <mesh filename="package://rr_openrover_description/meshes/4WD_Rover/LeftRearWheel.stl" scale="0.001 0.001 0.001"/>
+      </geometry>
+      <material name="dark"/>
+    </visual>
+    <collision>
+      <origin xyz="0 0 0" rpy="${pi / 2} 0 0"/>
+      <geometry>
+        <cylinder length="0.07" radius="0.127"/>
+      </geometry>
+    </collision>
+    <inertial>
+      <origin xyz="0 0 0" rpy="0 0 0"/>
+      <mass value="0.25" />
+      <inertia ixx="7.750e-6"
+               ixy="0.0" iyy="4.546-6"
+               ixz="0.0" iyz="1.478e-8" izz="4.545-6" />
+    </inertial>
+  </link>
+  <joint name="left_rear_wheel_joint" type="continuous">
+    <parent link="chassis_link"/>
+    <child link="left_rear_wheel_link"/>
+    <origin xyz="-0.284 0.18 0" rpy="0 0 0"/>
+    <axis xyz="0 1 0"/>
+  </joint>
+  <link name="right_rear_wheel_link">
+    <visual>
+      <origin xyz="0.284 0.18 0" rpy="${pi / 2} 0 ${pi / 2}"/>
+      <geometry>
+        <mesh filename="package://rr_openrover_description/meshes/4WD_Rover/RightRearWheel.stl" scale="0.001 0.001 0.001"/>
+      </geometry>
+      <material name="dark"/>
+    </visual>
+    <collision>
+      <origin xyz="0 0 0" rpy="${pi / 2} 0 0"/>
+      <geometry>
+        <cylinder length="0.07" radius="0.127"/>
+      </geometry>
+    </collision>
+    <inertial>
+      <origin xyz="0 0 0" rpy="0 0 0"/>
+      <mass value="0.25" />
+      <inertia ixx="7.750e-6"
+               ixy="0.0" iyy="4.546-6"
+               ixz="0.0" iyz="1.478e-8" izz="4.545-6" />
+    </inertial>
+  </link>
+  <joint name="right_rear_wheel_joint" type="continuous">
+    <parent link="chassis_link"/>
+    <child link="right_rear_wheel_link"/>
+    <origin xyz="-0.284 -0.18 0" rpy="0 0 0"/>
+    <axis xyz="0 1 0"/>
+  </joint>
+<!--<xacro:include filename="$(find rr_openrover_description)/urdf/accessories.urdf.xacro" />-->
 </robot>
